File: OpenTelemetry.sch (KiCad schematic (older format))
At the start: 23 parts, among them J1 Conn_ARM_JTAG_SWD_10, J2 Conn_01x09, J3 USB_B_Micro, U1 Adafruit-GPS, U2 TCAN1042xV, U3 STM32F072RBTx, U4 Adafruit-BNO055, U5 RFD900x, U6 HY28B

Commit message: V1 finished
Parts:
- removed U6: HY28B, JohnLib:HY28B, symbol JohnLib:HY28B
- added C11: 220uF, Capacitor_SMD:CP_Elec_8x10, symbol Device:C_Small
- added C12, C13: 100nF, Capacitor_SMD:C_0603_1608Metric, symbol Device:C_Small
- added D1: D_Schottky, Diode_SMD:D_SMA, symbol Device:D_Schottky
- added J4: Conn_01x15_Female, Connector_PinHeader_2.54mm:PinHeader_1x15_P2.54mm_Vertical, symbol Connector:Conn_01x15_Female
- added L2: 33uH, Inductor_SMD:L_TDK_SLF7045, symbol Device:L
- added U6: LM2596S-5, Package_TO_SOT_SMD:TO-263-5_TabPin3, symbol Regulator_Switching:LM2596S-5
Connections:
- net +3V3: now also J4.3 (Pin_3); no longer J2.5 (Pin_5)
- net +5V: now also C11.1, C12.1, C13.1, J4.1 (Pin_1), L2.1, U6.4 (FB); no longer J2.6 (Pin_6)
- net GND: now also J2.4 (Pin_4), C11.2, C12.2, C13.2, D1.2 (A), J4.2 (Pin_2), U6.3 (GND), U6.5 (~ON~/OFF)
- net LCD_CS: now also U3.3 (PC14), J4.8 (Pin_8)
- net LCD_RST: now also U3.38 (PC7), J4.9 (Pin_9)
- net LCD_SCK: now also J4.5 (Pin_5)
- net LCD_SDI: now also J4.7 (Pin_7)
- net LCD_SDO: now also J4.6 (Pin_6)
- net TP_X+: now reaches U3.2 (PC13)
- net TP_X+: now also J4.15 (Pin_15)
- net LITE: now reaches U3.37 (PC6)
- net LITE: now also J4.4 (Pin_4)
- net LCD_WAIT: now reaches U3.39 (PC8)
- net LCD_WAIT: now also J4.10 (Pin_10)
- net LCD_INT: now reaches U3.40 (PC9)
- net LCD_INT: now also J4.11 (Pin_11)
- net TP_Y+: now reaches U3.51 (PC10)
- net TP_Y+: now also J4.12 (Pin_12)
- net TP_Y-: now reaches U3.52 (PC11)
- net TP_Y-: now also J4.13 (Pin_13)
- net TP_X-: now reaches U3.53 (PC12)
- net TP_X-: now also J4.14 (Pin_14)
- net MISO: no longer names the net of U3.56 (PB4)
- net MOSI: no longer names the net of U3.57 (PB5)
- net SCK: no longer names the net of U3.55 (PB3)
- new net Batt+: J2.5 (Pin_5), U6.1 (VIN)
- new net Reg_Out: D1.1 (K), L2.2, U6.2 (OUT)
- no-connect marks 24 -> 20
